File: hw/sensors.kicad_sch (KiCad schematic)
At the start: 25 parts, among them U2 TSOP75438WTT, U3 INMP441ACEZ-R7

Commit message: Version 1.1 changes
Parts:
- removed R5, R6, R7: 510, Resistor_SMD:R_0805_2012Metric_Pad1.20x1.40mm_HandSolder, symbol Device:R
- removed TP4, TP5, TP6, TP7: TestPoint, TestPoint:TestPoint_Pad_1.0x1.0mm, symbol Connector:TestPoint
- R3: renamed from R2; value 10k -> 20k
- R4: renamed from R3; value 10k -> 20k
- R5: renamed from R4; value 10k -> 20k
- R9: value 10k -> 20k
Connections:
- net TB1: now also SW1.1
- net TB2: now also SW2.1
- net TB3: now also SW3.1
Other:
- moved on the sheet: SW1, SW2, SW3
